File: Hardware/LoraWan_Prototype_V1/Lorawan_Prototype_v1/Lorawan_Prototype_v1.kicad_sch (KiCad schematic)
At the start: 57 parts, among them J1 USB_B_Micro, J2 Conn_02x05_Odd_Even, J3 Conn_01x06, Q1 BC846, SW1 SW_SPDT, U1 USBLC6-2SC6, U2 BQ27441-G1, U3 STM32F103CBT6, U4 ZXMP6A13FTA, U5 BQ27441-G1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

Commit message: added 3.3v regulator and other suppport schematics- still a work in progress
Parts:
- removed C3: 1.0uF, sparkfun-battery-babysitter:0603-CAP, symbol sparkfun-battery-babysitter-eagle-import:1.0UF-16V-10%(0603)
- removed C7: 0.47uF, sparkfun-battery-babysitter:0603-CAP, symbol sparkfun-battery-babysitter-eagle-import:CAP0603-CAP
- removed R3: 0.01, sparkfun-battery-babysitter:1206, symbol sparkfun-battery-babysitter-eagle-import:RESISTOR1206
- removed U5: BQ27441-G1, sparkfun-battery-babysitter:PDSO-N12, symbol sparkfun-battery-babysitter-eagle-import:BQ27441-G1
- added C22, C23: 100nF, symbol Device:C
- added C24: 22uF, Capacitor_SMD:C_0603_1608Metric, symbol Device:C
- added C3, C7: 0.1uF, Capacitor_SMD:C_0603_1608Metric, symbol Device:C
- added D3: LED_YELLOW, symbol Device:LED
- added H1, H2, H3, H4: MountingHole_Pad, MountingHole:MountingHole_3mm_Pad_Via, symbol Mechanical:MountingHole_Pad
- added L2: L, symbol Device:L
- added R3: 1k, Resistor_SMD:R_0603_1608Metric, symbol Device:R
- added U10: BME280, Package_LGA:Bosch_LGA-8_2.5x2.5mm_P0.65mm_ClockwisePinNumbering, symbol Sensor:BME280
- added U5: AMS1117-3.3, Package_TO_SOT_SMD:SOT-223-3_TabPin2, symbol Regulator_Linear:AMS1117-3.3
- BT1: footprint BAT_MS621FE-FL11E -> MS621FE-FL11E:BAT_MS621FE-FL11E
- C12: footprint (none) -> Inductor_SMD:L_0805_2012Metric
Connections:
- net +3.3V: now also C22.1, C23.1, C24.1, C7.1, L2.2, U10.2 (CSB), U10.6 (VDDIO), U10.8 (VDD)
- net +5V: now also C3.1, U5.3 (VI)
- net GND: now also U2.13 (PAD), C22.2, C23.2, C24.2, C3.2, C7.2, D3.1 (K), U10.1 (GND), U10.5 (SDO), U10.7 (GND), U5.1 (GND)
- net SCL: now also U10.4 (SCK)
- net SDA: now also U10.3 (SDI)
- new net: L2.1, R3.1, U5.2 (VO)
- new net: D3.2 (A), R3.2
Other:
- note added: "3.3V REGULATOR"
- note added: "environmental sensors"
- note removed: "BQ27441-G1 Fuel Gauge"
- note removed: "I2C ADDR: 0x55"
- note removed: "VDD is 1.8V generated internally"
- moved on the sheet: BT1, C1, C14, C15, C16, C18, C2, C20, C21, D1, D2, J3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
